File: starbiebutporro.kicad_pcb (KiCad board)
At the start: 2 copper layers, 99.2 x 127 mm, 10 parts, among them J1 Conn_01x04_Pin, J2 Conn_01x08_Pin, SW1 SW_Push, SW2 SW_Push, SW4 SW_SPST, U1 XIAO-ESP32-C3-SMD, U2 DHT11

Commit message: Add files via upload
Parts:
- removed BT1: Battery_Cell, Battery:BatteryHolder_Keystone_1042_1x18650
- removed F1: Fuse, Fuse:Fuse_1206_3216Metric
- removed SW4: SW_SPST, Button_Switch_SMD:SW_DIP_SPSTx01_Slide_6.7x4.1mm_W6.73mm_P2.54mm_LowProfile_JPin
Connections:
- U1 pad 21: /+VBAT -> unconnected-(U1-VBAT-Pad21)
- U1 pad 22: /-VBAT -> unconnected-(U1-GND-Pad22)
Routing:
- net /-VBAT: track 89.6 -> 0.00 mm, vias 1 -> 0
- net Net-(BT1-+): track 55.9 -> 0.00 mm
- net /+VBAT: track 36.4 -> 0.00 mm, vias 1 -> 0
- net Net-(SW4-A): track 9.68 -> 0.00 mm
Other:
- board size 99.2 x 127 mm -> 99.2 x 87.8 mm
