File: starbiebutporro.kicad_sch (KiCad schematic)
At the start: 10 parts, among them J1 Conn_01x04_Pin, J2 Conn_01x08_Pin, SW1 SW_Push, SW2 SW_Push, SW4 SW_SPST, U1 XIAO-ESP32-C3-SMD, U2 DHT11

Commit message: Add files via upload
Parts:
- removed BT1: Battery_Cell, Battery:BatteryHolder_Keystone_1042_1x18650, symbol Device:Battery_Cell
- removed F1: Fuse, Fuse:Fuse_1206_3216Metric, symbol Device:Fuse
- removed SW4: SW_SPST, Button_Switch_SMD:SW_DIP_SPSTx01_Slide_6.7x4.1mm_W6.73mm_P2.54mm_LowProfile_JPin, symbol Switch:SW_SPST
Connections:
- net +VBAT: no longer names the net of U1.21 (VBAT)
- net -VBAT: no longer names the net of U1.22 (GND)
- no-connect marks 16 -> 18
